File: hardware/kicad/HPVE_Controller.kicad_pcb (KiCad board)
At the start: 2 copper layers, 124 x 94 mm, 105 parts, among them U1 74HC595, U10 RP2040_Pico, U101 TC4427ACOA, U102 TC4427ACOA, U103 TC4427ACOA, U104 TC4427ACOA, U105 TC4427ACOA, U106 TC4427ACOA, U107 TC4427ACOA, U108 TC4427ACOA, U109 TC4427ACOA, U110 TC4427ACOA, U111 TC4427ACOA, U112 TC4427ACOA, U113 TC4427ACOA, U114 TC4427ACOA, U115 TC4427ACOA, U116 TC4427ACOA, U117 TC4427ACOA, U118 TC4427ACOA, U119 TC4427ACOA, U120 TC4427ACOA, U121 TC4427ACOA, U122 TC4427ACOA, U123 TC4427ACOA, U124 TC4427ACOA, U125 TC4427ACOA, U126 TC4427ACOA, U127 TC4427ACOA, U128 TC4427ACOA, U129 TC4427ACOA, U130 TC4427ACOA, U131 TC4427ACOA, U132 TC4427ACOA, U2 74HC595, U3 74HC595, U4 74HC595, U5 74HC595, U6 74HC595, U7 74HC595, U8 74HC595

Commit message: feat(hardware): 7-hour session 2 sprint - 2,448 tracks & 329 vias routed, 116 shorts eliminated, edge clearance fixed, 124 XP locked
Routing:
- net GND: track 510.5 -> 0.00 mm
- net /TC4427_Driver_Bank/GND: track 0.00 -> 276.1 mm, vias 0 -> 5
- net DRV_14: track 55.2 -> 192.8 mm, vias 0 -> 6
- net DRV_8: track 72.9 -> 195.9 mm, vias 0 -> 3
- net DRV_21: track 66.9 -> 187.1 mm, vias 0 -> 8
- net /Shift_Register_Cascade/SPI_SCK: track 0.00 -> 119.6 mm
- net SIG_61: track 73.3 -> 179.8 mm, vias 0 -> 5
- net SIG_44: track 66.4 -> 170.4 mm, vias 0 -> 7
- net DRV_3: track 43.5 -> 139.9 mm, vias 0 -> 12
- net DRV_15: track 61.5 -> 154.9 mm, vias 0 -> 7
- net DRV_9: track 79.2 -> 169.3 mm, vias 0 -> 6
- net SIG_63: track 74.8 -> 154.1 mm, vias 0 -> 4
- net DRV_16: track 67.1 -> 141.2 mm, vias 0 -> 4
- net DRV_22: track 72.6 -> 0.00 mm
- net SIG_46: track 67.9 -> 0.00 mm
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